File: GR8RAM.kicad_pcb (KiCad board)
At the start: 4 copper layers, 107.6 x 59.8 mm, 44 parts, among them J1 AppleIIBus, J2 JTAG, U1 EPM7128SL84, U5 39F040

Commit message: Release candidate PCB
Parts:
- removed the C12 at (49.3, 128.3)
- removed the C12 at (149.7, 89.5)
- removed the C13 at (94.8, 128.3)
- removed the C13 at (174.5, 79.1)
- removed FD1, FD2, FD3, FD4, FD5: Fiducial, stdpads:Fiducial
- removed R6, R7: 100, stdpads:R_0805
- removed REF** (x4): SOJ-24-26-300mil, stdpads:SOJ-24-26-300mil
- added C12: 100n, stdpads:C_0805, F.Cu at (119.0, 83.8)
- added C13: 100n, stdpads:C_0805, F.Cu at (136.3, 128.3)
- added C21: 100n, stdpads:C_0805, F.Cu at (76.2, 125.3)
- added C22: 100n, stdpads:C_0805, F.Cu at (120.2, 126.2)
- added FID1: Fiducial, stdpads:Fiducial, F.Cu at (143.0, 82.4)
- added FID2: Fiducial, stdpads:Fiducial, F.Cu at (40.5, 96.1)
- added FID3: Fiducial, stdpads:Fiducial, F.Cu at (54.2, 82.4)
- added FID4: Fiducial, stdpads:Fiducial, F.Cu at (143.0, 129.5)
- added FID5: Fiducial, stdpads:Fiducial, F.Cu at (40.5, 129.5)
- added JP1: Mode, Connector_PinHeader_2.54mm:PinHeader_1x02_P2.54mm_Vertical_SMD_Pin1Left, F.Cu at (139.7, 91.4)
- added R1: 100, stdpads:R_0805, F.Cu at (102.9, 128.3)
- added R2: 100, stdpads:R_0805, F.Cu at (105.4, 128.3)
- added R3: 100, stdpads:R_0805, F.Cu at (108.0, 128.3)
- added U2: 39F040, stdpads:PLCC-32_SMDSocket, F.Cu at (50.8, 111.8)
- added U3: AS4C4M4, stdpads:SOP-24-26-300mil, F.Cu at (85.1, 114.3)
- added U4: AS4C4M4, stdpads:SOP-24-26-300mil, F.Cu at (85.1, 94.0)
- added U6: AS4C4M4, stdpads:SOP-24-26-300mil, F.Cu at (71.1, 94.0)
- C14: value 5p -> 33u; footprint stdpads:C_0805 -> stdpads:CP_EIA-3528
- C15: value 100n -> 33u; footprint stdpads:C_0805 -> stdpads:CP_EIA-3528
- C18: value 33u -> 100n; footprint stdpads:CP_EIA-3528 -> stdpads:C_0805
- J2: footprint Connector_IDC:IDC-Header_2x05_P2.54mm_Vertical -> stdpads:IDC_SMD_2x05_P2.54mm_Vertical
- R5: value 100 -> 820
- U5: value 39F040 -> AS4C4M4; footprint stdpads:PLCC-32_SMDSocket -> stdpads:SOP-24-26-300mil
- moved C10 153.7 mm to (89.3, 83.8), turned to 180 degrees
- moved C8 148.5 mm to (71.4, 128.3)
- moved C7 143.9 mm to (89.3, 124.5), turned to 180 degrees
- moved C6 99.6 mm to (132.1, 98.2), turned to 90 degrees
- moved C16 95.7 mm to (55.1, 92.8), turned to 180 degrees
- moved C19 91.2 mm to (75.3, 128.3), turned to 180 degrees
- moved C9 81.2 mm to (126.4, 124.5)
- moved C20 56.7 mm to (120.2, 128.3), turned to 180 degrees
- moved R5 54.1 mm to (108.3, 83.8), turned to 180 degrees
- moved C15 50.5 mm to (134.9, 83.8), turned to 0 degrees
- moved U5 45.8 mm to (71.1, 114.3), turned to 180 degrees
- moved C5 44.0 mm to (98.2, 83.8), turned to 180 degrees
- moved C11 43.3 mm to (112.6, 83.8)
- moved C14 38.1 mm to (140.3, 125.1), turned to 180 degrees
- moved C1 35.2 mm to (75.3, 104.1), turned to 180 degrees
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Connections:
- C14 pad 1: Net-(C14-Pad1) -> +5V
- C18 pad 1: GND -> +5V
- C19 pad 2: Net-(C19-Pad2) -> GND
- C20 pad 1: Net-(C19-Pad2) -> GND
- J1 pad 23: /INTout -> /INTin
- J1 pad 24: /DMAout -> /DMAin
- R5 pad 1: /PHI0r -> +5V
- R5 pad 2: /PHI0 -> /~MODE~
- U1 pad 10: /~INH~ -> /A9
- U1 pad 11: /SYNC -> /A10
- U1 pad 12: Net-(U1-Pad12) -> /A11
- U1 pad 15: /RAMROM~CS~ -> /A12
- U1 pad 16: /RAMCS -> /A13
- U1 pad 17: /ROM~OE~ -> /A14
- U1 pad 18: /ROM~WE~ -> /A15
- U1 pad 2: /PHI1 -> /PHI1r
- U1 pad 20: Net-(U1-Pad20) -> /R~W~
- U1 pad 21: Net-(U1-Pad21) -> /~DEVSEL~
- U1 pad 22: /D7 -> /~INH~
- U1 pad 24: /D6 -> /~IOSTRB~
- U1 pad 25: /D5 -> /D7
- U1 pad 27: /D4 -> /D6
- U1 pad 28: /D3 -> /D5
- U1 pad 29: /D2 -> /D4
- U1 pad 30: /D1 -> Net-(U1-Pad30)
- U1 pad 31: /D0 -> Net-(U1-Pad31)
- U1 pad 33: /A15 -> /D3
- U1 pad 34: /A14 -> /D2
- U1 pad 35: /A13 -> /D1
- U1 pad 36: /A12 -> /D0
- U1 pad 37: /A11 -> Net-(U1-Pad37)
- U1 pad 39: /A10 -> /~CAS~0
- U1 pad 4: /PHI0 -> /A6
- U1 pad 40: /A9 -> /~CAS~1
- U1 pad 41: /A8 -> /R~CS~
- U1 pad 44: /A7 -> /~MODE~
- U1 pad 45: /A6 -> /R~OE~
- U1 pad 46: /A5 -> /RA9
- U1 pad 48: /A4 -> /RA10
- U1 pad 49: /A3 -> /RA3
- U1 pad 5: /R~W~ -> /A7
- U1 pad 50: /A2 -> /RA2
- U1 pad 51: /A1 -> /RA5
- U1 pad 52: /A0 -> /RA0
- U1 pad 54: /RA0 -> /RA1
- U1 pad 55: /RA1 -> /RA4
- U1 pad 56: /RA2 -> /RA7
- U1 pad 57: /RA3 -> /RA6
- U1 pad 58: /RA4 -> /RA8
- U1 pad 6: /~IOSEL~ -> /Q3r
- U1 pad 60: /RA5 -> /~RAS~
- U1 pad 61: /RA6 -> /RD7
- U1 pad 63: /RA7 -> /RD5
- U1 pad 64: /RA8 -> /RD6
- U1 pad 65: /RA9 -> /RD4
- U1 pad 67: /RA10 -> /R~WE~
- U1 pad 68: /RA11 -> /RD3
- U1 pad 69: /RA12 -> /RD2
- U1 pad 70: /RA13 -> /RD1
- U1 pad 73: /RA14 -> /RD0
- U1 pad 74: /RA15 -> /~IOSEL~
- U1 pad 75: /RA16 -> /A0
- U1 pad 76: /RA17 -> /A1
- U1 pad 77: /RA18 -> /A2
- U1 pad 79: /RA19 -> /A3
- U1 pad 8: /~DEVSEL~ -> /PHI0r
- U1 pad 80: /Q3 -> /A4
- U1 pad 81: Net-(U1-Pad81) -> /A5
- U1 pad 83: /7M -> /7Mr
- U1 pad 84: /7M -> /7Mr
- U1 pad 9: /~IOSTRB~ -> /A8
- U5 pad 1: /RA18 -> +5V
- U5 pad 10: /A2 -> /RA2
- U5 pad 11: /A1 -> /RA3
- U5 pad 12: /A0 -> /RA10
- U5 pad 13: /RD5 -> +5V
- U5 pad 14: /RD6 -> GND
- U5 pad 15: /RD4 -> /RA9
- U5 pad 16: GND -> /RA8
- U5 pad 17: /RD7 -> /RA6
- U5 pad 18: /RD1 -> /RA7
- U5 pad 19: /RD2 -> /RA4
- U5 pad 2: /RA16 -> /RD1
- U5 pad 21: /RD3 -> /RA1
- U5 pad 22: /RAMROM~CS~gb -> GND
- U5 pad 23: /A10 -> /~CAS~1
- U5 pad 24: /ROM~OE~ -> /RD2
- U5 pad 25: /A11 -> /RD0
- U5 pad 26: /A9 -> GND
- U5 pad 3: /RA15 -> /RD3
- U5 pad 4: /RA12 -> /R~WE~
- U5 pad 5: /A7 -> /~RAS~
- U5 pad 6: /A6 -> (no net)
- U5 pad 8: /A4 -> /RA0
- U5 pad 9: /A3 -> /RA5
Routing:
- net +5V: track 13.2 -> 157.1 mm, vias 6 -> 77
- net /RA0: track 0.00 -> 115.4 mm
- net GND: track 22.6 -> 136.7 mm, vias 89 -> 441
- net /RA5: track 0.00 -> 112.5 mm
- net /R~CS~: track 0.00 -> 109.7 mm, vias 0 -> 2
- net /A9: track 17.0 -> 125.5 mm, vias 0 -> 2
- net /A7: track 16.5 -> 124.6 mm, vias 0 -> 2
- net /A8: track 16.5 -> 124.0 mm, vias 0 -> 2
- net /RA1: track 0.00 -> 106.4 mm
- net /A6: track 15.9 -> 120.2 mm, vias 0 -> 2
- net /R~WE~: track 0.00 -> 102.0 mm, vias 0 -> 4
- net /RA2: track 0.00 -> 101.2 mm
- net /RA4: track 0.00 -> 100.7 mm
- net /RA3: track 0.00 -> 98.8 mm
- net /RA7: track 0.00 -> 97.4 mm
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Other:
- outline, holes or cut-outs redrawn
- rule solder_mask_min_width: 0.1524 -> 0.127
- board text added: "4204A"
- board text added: "8 MB RAM"
- board text removed: "4205A"
- board text removed: "8M RAM"

Commit message: Submitted to JLCPCB
Routing:
- net GND: vias 441 -> 444
Changed lines of the file:
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@@
     (thickness 1.6)
     (drawings 30)
-    (tracks 1902)
+    (tracks 1904)
     (zones 0)
     (modules 46)
@@
   (via (at 123.317 127.381) (size 0.6) (drill 0.3) (layers F.Cu B.Cu) (net 2))
   (via (at 122.809 121.92) (size 0.6) (drill 0.3) (layers F.Cu B.Cu) (net 2))
+  (via (at 87.757 127.508) (size 0.6) (drill 0.3) (layers F.Cu B.Cu) (net 2))
+  (via (at 85.852 122.809) (size 0.6) (drill 0.3) (layers F.Cu B.Cu) (net 2))
+  (via (at 78.105 114.427) (size 0.6) (drill 0.3) (layers F.Cu B.Cu) (net 2))
   (segment (start 88.9 130.81) (end 88.9 135.382) (width 0.1524) (layer F.Cu) (net 3))
   (segment (start 88.9 130.81) (end 89.83981 129.87019) (width 0.1524) (layer F.Cu) (net 3))
@@
   (segment (start 110.49 111.328934) (end 106.40057 115.418364) (width 0.1524) (layer B.Cu) (net 20))
   (via (at 99.06 101.6) (size 0.6) (drill 0.3) (layers F.Cu B.Cu) (net 21))
-  (segment (start 92.07728 107.18572) (end 97.663 101.6) (width 0.1524) (layer B.Cu) (net 21))
   (segment (start 92.07728 107.19028) (end 92.07728 107.18572) (width 0.1524) (layer B.Cu) (net 21))
   (segment (start 92.075 107.188) (end 92.07728 107.19028) (width 0.1524) (layer B.Cu) (net 21))
-  (segment (start 97.663 101.6) (end 99.06 101.6) (width 0.1524) (layer B.Cu) (net 21))
-  (segment (start 80.41648 118.84652) (end 92.075 107.188) (width 0.1524) (layer B.Cu) (net 21))
-  (segment (start 61.94318 118.84652) (end 80.41648 118.84652) (width 0.1524) (layer B.Cu) (net 21))
   (segment (start 56.3625 114.3) (end 57.785 114.3) (width 0.1524) (layer F.Cu) (net 21))
   (segment (start 57.785 114.68834) (end 61.94318 118.84652) (width 0.1524) (layer B.Cu) (net 21))
@@
   (segment (start 124.46 120.015) (end 123.13919 121.33581) (width 0.1524) (layer F.Cu) (net 21))
   (segment (start 124.46 118.49) (end 124.46 120.015) (width 0.1524) (layer F.Cu) (net 21))
+  (segment (start 99.06 101.6) (end 97.766802 101.6) (width 0.1524) (layer B.Cu) (net 21))
+  (segment (start 97.766802 101.6) (end 80.520282 118.84652) (width 0.1524) (layer B.Cu) (net 21))
+  (segment (start 80.520282 118.84652) (end 61.94318 118.84652) (width 0.1524) (layer B.Cu) (net 21))
   (via (at 76.2 129.54) (size 0.8) (drill 0.4) (layers F.Cu B.Cu) (net 22))
   (segment (start 76.2 128.27) (end 76.2 129.54) (width 0.762) (layer F.Cu) (net 22))

Commit message: New schematic revision
Parts:
- C1, C10, C11, C12, C13, C17, C18, C19, C2, C20, C21, C22, C3, C4, C5, C6, C7, C8, C9: value 100n -> 2u2
- C14, C15, C16: value 33u -> DNP
- R4: value 100 -> 15
- R5: value 820 -> 22k
- U2: value 39F040 -> 512Kx8 Flash
- U3, U4, U5, U6: value AS4C4M4 -> 4Mx4 DRAM
Connections:
- net /SYNC renamed /VIDSYNC
- net Net-(U1-Pad30) renamed /PHI1out
- net Net-(U1-Pad31) renamed /C7Mout
