File: GR8RAM.kicad_pcb (KiCad board)
At the start: 4 copper layers, 99.9 x 59.8 mm, 122 parts, among them J1 AppleIIBus, J2 JTAG, J3 DC in, J4 JTAG, J5 JTAG, Q1 AO3401A, U1 EPM240T100C5N, U10 LM393D, U11 74LVC1G125GW, U12 74LVC1G125GW, U13 25M, U14 74LVC1G125GW, U15 74LVC1G125GW, U16 74LVC1G125GW, U17 74LVC1G125GW, U18 74LVC1G125GW, U19 74LVC1G125GW, U2 W9825, U20 74LVC1G125GW, U22 74LVC1G125GW, U3 W25Q128JVSIQ, U4 74AHC245PW, U5 74AHC245PW, U6 74AHC245PW, U7 LM393D, U8 XC6206P332MR, U9 74AHC245PW

Commit message: idk
Parts:
- added C17: 1n, stdpads:C_0603, F.Cu at (131.4, 106.3)
- C41: value 22n -> 2u2
- D1, D3: value SS14 -> SS34
- R18: value 22k -> 100k
- moved C11 3.45 mm to (132.3, 102.1), turned to 180 degrees
Routing:
- net +5V: track 223.5 -> 235.8 mm, vias 5 -> 6
- net Net-(C17-Pad2): track 10.6 -> 13.1 mm
- net /~Menu~: track 100.7 -> 98.8 mm
- net +3V3: track 156.0 -> 154.5 mm, vias 113 -> 114
- added copper zone on F.Cu, net Net-(C39-Pad1)
- removed copper zone on F.Cu, net Net-(C17-Pad2)

Commit message: Works?
Parts:
- removed C17, C39: 1n, stdpads:C_0603
- removed C38, C40: 22n, stdpads:C_0603
- removed C41: 2u2, stdpads:C_0603
- removed C5, C6: 10u, stdpads:C_0805
- removed D1, D3: SS34, stdpads:D_SMA
- removed D2: SMBJ5.0A, stdpads:D_SMB
- removed F1: nSMD050-16V, stdpads:BelFuse_1206
- removed FB1: GZ2012D101TF, stdpads:Murata_BLM21
- removed J3: DC in, stdpads:BOOMELE_DC-005_DC_5.5-2.0MM
- removed Q1: AO3401A, stdpads:SOT-23
- removed R1, R20, R21, R23, R24, R25, R26, R27: 33, stdpads:R_0603
- removed R10, R15, R16, R2, R4: 2k2, stdpads:R_0603
- removed R11: 330, stdpads:R_0603
- removed R12: 1k, stdpads:R_0805
- removed R13: DNP, stdpads:R_0805
- removed R14, R17, R6: 1k, stdpads:R_0603
- removed R18: 100k, stdpads:R_0603
- removed R3: 2k7, stdpads:R_0603
- removed R30, R5, R8: 1M, stdpads:R_0603
- removed R7: 820, stdpads:R_0603
- removed R9: 1k2, stdpads:R_0603
- removed RN4: 4x10k, stdpads:R4_0402
- removed U10, U7: LM393D, stdpads:SOIC-8_3.9mm
- removed U11, U12, U15, U17, U18, U19, U20, U22: 74LVC1G125GW, stdpads:SOT-353
- added REF**: SW_DIP_SPSTx02_Slide_DSHP02TS_P1.27mm, stdpads:SW_DIP_SPSTx02_Slide_DSHP02TS_P1.27mm, F.Cu at (135.8, 95.7)
- moved C44 60.9 mm to (69.0, 100.7)
- moved C9 27.5 mm to (112.2, 90.8), turned to 0 degrees
- moved C43 17.9 mm to (104.8, 112.2), turned to 0 degrees
- moved C36 17.8 mm to (133.3, 114.9), turned to 0 degrees
- moved C37 13.4 mm to (137.7, 111.9), turned to 0 degrees
- moved C11 9.82 mm to (133.3, 111.9), turned to 0 degrees
- moved C12 7.49 mm to (141.3, 114.6), turned to 0 degrees
- moved C42 3.98 mm to (117.8, 122.1), turned to 90 degrees
- moved R22 1.00 mm to (115.8, 124.2)
- moved U14 1.00 mm to (115.7, 121.8)
Connections:
- C7 pad 1: Vin -> +5V
- C8 pad 1: Vin -> +5V
- J1 pad 23: /INTout -> /INTin
- J1 pad 24: /DMAout -> /DMAin
- U8 pad 3: Vin -> +5V
- U9 pad 1: /Adir -> +3V3
Routing:
- net +5V: track 235.8 -> 45.6 mm, vias 6 -> 3
- net /~Menu~: track 98.8 -> 0.00 mm, vias 2 -> 0
- net /DMA~OE~: track 79.1 -> 0.00 mm, vias 3 -> 0
- net /RINTout: track 77.5 -> 0.00 mm, vias 2 -> 0
- net /~BOD~: track 77.2 -> 0.00 mm, vias 2 -> 0
- net GND: track 235.8 -> 160.7 mm, vias 440 -> 410
- net /RDMAout: track 74.8 -> 0.00 mm, vias 2 -> 0
- net /~PreBOD~: track 70.3 -> 0.00 mm, vias 2 -> 0
- net /Adir: track 57.9 -> 0.00 mm, vias 3 -> 0
- net /NMI~OE~: track 55.5 -> 0.00 mm, vias 2 -> 0
- net /DMAin: track 51.0 -> 0.00 mm, vias 4 -> 0
- net /IRQ~OE~: track 50.6 -> 0.00 mm, vias 2 -> 0
- net /RDY~OE~: track 48.3 -> 0.00 mm, vias 2 -> 0
- net /INTin: track 46.9 -> 0.00 mm, vias 4 -> 0
- net /INH~OE~: track 45.8 -> 0.00 mm, vias 2 -> 0
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- removed copper zone on F.Cu, net Net-(C39-Pad1)
- removed copper zone on F.Cu, net Net-(C40-Pad1)

Commit message: idk
Parts:
- removed C36, C37, C8: 10u, stdpads:C_0805
- removed C9: 2u2, stdpads:C_0603
- removed R19: 1k, stdpads:R_0603
- removed REF**: SW_DIP_SPSTx02_Slide_DSHP02TS_P1.27mm, stdpads:SW_DIP_SPSTx02_Slide_DSHP02TS_P1.27mm
- added C5: 2u2, stdpads:C_0603, F.Cu at (113.7, 90.8)
- added SW1: FW, stdpads:SW_DIP_SPSTx02_Slide_DSHP02TS_P1.27mm, F.Cu at (135.8, 95.9)
- moved C12 29.7 mm to (123.7, 90.8), turned to 180 degrees
- moved C7 20.8 mm to (140.1, 124.2), turned to 90 degrees
- moved C10 18.8 mm to (132.8, 124.2)
- moved U8 18.8 mm to (136.2, 124.2)
- moved C11 12.7 mm to (130.3, 124.2), turned to 90 degrees
- moved RN5 0.15 mm to (69.1, 96.5)
Connections:
- net /DMA~OE~ renamed Net-(U1-Pad21)
- net /INH~OE~ renamed Net-(U1-Pad27)
- net /IRQ~OE~ renamed Net-(U1-Pad29)
- net /NMI~OE~ renamed Net-(U1-Pad26)
- net /RDMAout renamed Net-(U1-Pad18)
- net /RDY~OE~ renamed Net-(U1-Pad28)
- net /RINTout renamed Net-(U1-Pad20)
- net /RR~W~out renamed Net-(U1-Pad33)
- U1 pad 19: /Adir -> Net-(U1-Pad19)
- U1 pad 48: /RDMAin -> Net-(U1-Pad48)
- U1 pad 49: /RINTin -> Net-(U1-Pad49)
- U1 pad 95: /~BOD~ -> /FW1
- U1 pad 96: /~PreBOD~ -> /FW0
- U4 pad 1: /Adir -> +3V3
- U5 pad 11: /RINTin -> Net-(U5-Pad11)
- U5 pad 12: /RDMAin -> Net-(U5-Pad12)
- U5 pad 8: /DMAin -> GND
- U5 pad 9: /INTin -> GND
Routing:
- net /FW0: track 0.00 -> 56.0 mm, vias 0 -> 2
- net /FW1: track 0.00 -> 53.1 mm, vias 0 -> 2
- net +3V3: track 127.4 -> 148.5 mm, vias 97 -> 113
- net /RINTin: track 17.8 -> 0.00 mm
- net /RDMAin: track 17.6 -> 0.00 mm
- net GND: track 160.7 -> 176.4 mm, vias 410 -> 456
- net /INTin: track 0.00 -> 8.38 mm, vias 0 -> 1
- net /DMAin: track 0.00 -> 8.38 mm, vias 0 -> 2
- net +5V: track 45.6 -> 41.1 mm
- net /~RES~: track 29.3 -> 27.2 mm
- net /MOSI: track 97.6 -> 96.8 mm, vias 2 -> 1
- net /Ddir: track 27.9 -> 27.0 mm
- net /FD2: track 48.9 -> 49.5 mm
- net (no net): vias 1 -> 0
- added copper zone on F.Cu, net +5V
Other:
- board text added: "1 MB RAMFactor"
- board text added: "1 MB Slinky"
- board text added: "16 MB RAMFactor*"
- board text added: "8 MB RAMFactor"
- board text added: "Firmware Select:"
