File: GR8RAM.sch (KiCad schematic (older format))
At the start: 46 parts, among them J1 AppleIIBus, J2 JTAG, U1 EPM7128SL84, U2 39F040, U3 AS4C4M4, U4 AS4C4M4, U5 AS4C4M4, U6 AS4C4M4

Commit message: New schematic revision
Parts:
- C1, C10, C11, C12, C13, C17, C18, C19, C2, C20, C21, C22, C3, C4, C5, C6, C7, C8, C9: value 100n -> 2u2
- C14, C15, C16: value 33u -> DNP
- R4: value 1 -> 15
- R5: value 4k7 -> 22k
- U1: symbol stdparts:EPM7128SL84 -> GW_PLD:EPM7128SL84
- U2: value 39F040 -> 512Kx8 Flash; symbol stdparts:39F040 -> GW_RAM:Flash-512Kx8-PLCC-32
- U3, U4, U5, U6: value AS4C4M4 -> 4Mx4 DRAM; symbol stdparts:AS4C4M4 -> GW_RAM:DRAM-4Mx4-SOP-24
