File: GR8RAM.sch (KiCad schematic (older format))
At the start: 98 parts, among them J1 AppleIIBus, J2 JTAG, J3 DC in, J4 JTAG, Q1 AO3401A, U1 EPM240T100C5N, U10 LM393, U12 74AHCT125, U13 25M, U14 74AHCT125, U16 74LVC1G04GW, U2 W9825, U3 MX29LV640EB, U4 74AHC245, U5 74AHC245, U6 74AHC245, U7 LM393, U8 AP2125, U9 74AHC245

Commit message: Fabbed
Parts:
- removed C17: 2u2, stdpads:C_0603, symbol Device:C_Small
- removed D1: M7, stdpads:D_SMA, symbol Device:D_Small_ALT
- removed U12, U14: 74AHCT125, stdpads:TSSOP-14_4.4x5mm_P0.65mm, symbol GW_Logic:74125
- removed U3: MX29LV640EB, stdpads:TSOP-I-48_18.4x12mm_P0.5mm, symbol GW_RAM:Flash-4Mx16-TSOP1-48
- added C42, C43, C44: 2u2, stdpads:C_0603, symbol Device:C_Small
- added D1: SS34, stdpads:D_SMA, symbol Device:D_Schottky_Small_ALT
- added J5: JTAG, Connector:Tag-Connect_TC2050-IDC-FP_2x05_P1.27mm_Vertical, symbol Connector_Generic:Conn_02x05_Odd_Even
- added R19: 1k, stdpads:R_0603, symbol Device:R_Small
- added R20, R21, R22, R23, R24, R25, R26, R27, R31: 33, stdpads:R_0603, symbol Device:R_Small
- added R28, R29: 22k, stdpads:R_0603, symbol Device:R_Small
- added R30: 1M, stdpads:R_0603, symbol Device:R_Small
- added RN5: 4x10k, stdpads:R4_0402, symbol Device:R_Pack04
- added U11, U12, U14, U15, U17, U18, U19, U20, U22: 74LVC1G125GW, stdpads:SOT-353, symbol GW_Logic:741G125GW
- added U3: W25Q128JVSIQ, stdpads:SOIC-8_5.3mm, symbol GW_RAM:SPIFlash-SO-8
- C38, C40, C41: value 10n -> 22n; LCSC Part C57112 -> C21122
- C39: value 10n -> 1n; LCSC Part C57112 -> C1588
- D3: value SS14 -> SS34; LCSC Part C2480 -> C8678
- F1: value nSMD035-16V -> nSMD050-16V; LCSC Part C70072 -> C70075
- FB1: value GZ2012D601TF -> GZ2012D101TF; LCSC Part C1017 -> C1015
- H2, H3, H4, H5, H6: symbol Mechanical:MountingHole_Pad -> Mechanical:MountingHole
- R1: value DNP -> 33; footprint stdpads:R_0805 -> stdpads:R_0603; LCSC Part (none) -> C23140
- R10, R15: value 1k -> 2k2; LCSC Part C21190 -> C4190
- R11: value 1k -> 330; LCSC Part C21190 -> C23138
- R13: value 100 -> DNP; LCSC Part C17408 -> (none)
- R2: value DNP -> 2k2; footprint stdpads:R_0805 -> stdpads:R_0603; LCSC Part (none) -> C4190
- R3: value 3k0 -> 2k7; LCSC Part C4211 -> C13167
- R7: value 1k -> 820; LCSC Part C21190 -> C23253
- R9: value 3k6 -> 1k2; LCSC Part C22980 -> C22765
- U10, U7: value LM393 -> LM393D
- U13: LCSC Part C32526 -> C669088
- U16: value 74LVC1G04GW -> 74LVC1G125GW; symbol GW_Logic:741G04GW -> GW_Logic:741G125GW; LCSC Part C10237 -> C12519
- U4, U5, U6, U9: value 74AHC245 -> 74AHC245PW
- U8: value AP2125 -> XC6206P332MR; LCSC Part C150715 -> C5446
Connections:
- net RW~OE~ is gone; now on net INH~OE~: U1.27 (IO1_27)
- net R~CS~ is gone; now on net RD0: U1.86 (IO2_86)
- net R~OE~ is gone; now on net SDQML: U1.85 (IO2_85)
- net +3V3: now also R2.1, C42.1, C43.1, C44.1, J5.2 (Pin_2), R28.1, RN5.5 (R4.2), RN5.6 (R3.2), RN5.7 (R2.2), RN5.8 (R1.2), U11.5 (Vcc), U12.5 (Vcc), U14.5 (Vcc), U15.5 (Vcc), U17.5 (Vcc), U18.5 (Vcc), U19.5 (Vcc), U20.5 (Vcc), U22.5 (Vcc), U3.8 (Vcc)
- net Adir: now also U20.1 (~OE~)
- net DMAin: now also RN4.1 (R1.1), U5.8 (A6); no longer R1.2, RN4.4 (R4.1), U5.9 (A7)
- net DMAout: now also R25.1; no longer R1.1
- net DMA~OE~: now also U1.21 (IO1_21), U15.1 (~OE~); no longer U1.30 (IO1_30)
- net Ddir: now also U1.17 (IO1_17); no longer U1.18 (IO1_18)
- net GND: now also C41.2, U16.1 (~OE~), U4.19 (~OE~), U6.19 (~OE~), U9.19 (~OE~), C42.2, C43.2, C44.2, J5.7 (Pin_7), R29.2, U11.2 (A), U11.3 (GND), U12.2 (A), U12.3 (GND), U14.2 (A), U14.3 (GND), U15.2 (A), U15.3 (GND), U17.2 (A), U17.3 (GND), U18.2 (A), U18.3 (GND), U19.2 (A), U19.3 (GND), U20.3 (GND), U22.2 (A), U22.3 (GND), U3.4 (GND); no longer C41.1, H2.1, H3.1, H4.1, H5.1, H6.1
- net INH~OE~: now also U22.1 (~OE~); no longer U1.33 (IO1_33)
- net INTin: now also RN4.4 (R4.1), U5.9 (A7); no longer R2.2, RN4.1 (R1.1), U5.8 (A6)
- net INTout: now also R26.1; no longer R2.1
- net IRQ~OE~: now also U11.1 (~OE~)
- net M+: now also C41.1, R30.2; no longer C41.2
- net NMI~OE~: now also U12.1 (~OE~)
- net PHI0: now also U5.4 (A2)
- net PHI1: no longer U5.4 (A2)
- net RA0: now also U1.100 (IO2_100); no longer U1.16 (IO1_16)
- net RA1: now also U1.98 (IO2_98); no longer U1.87 (IO2_87)
- net RA10: now also U1.14 (IO1_14/GCLK1); no longer U1.3 (IO1_3)
- net RA2: now also U1.97 (IO2_97); no longer U1.88 (IO2_88)
- net RA3: now also U1.4 (IO1_4); no longer U1.89 (IO2_89)
- net RA4: now also U1.1 (IO2_1); no longer U1.90 (IO2_90)
- net RA5: now also U1.2 (IO1_2); no longer U1.91 (IO2_91)
- net RA6: now also U1.3 (IO1_3); no longer U1.92 (IO2_92)
- net RA7: now also U1.6 (IO1_6); no longer U1.99 (IO2_99)
- net RA8: now also U1.7 (IO1_7); no longer U1.100 (IO2_100)
- net RA9: now also U1.8 (IO1_8); no longer U1.1 (IO2_1)
- net RD0: no longer U1.2 (IO1_2)
- net RD1: now also U1.87 (IO2_87); no longer U1.4 (IO1_4)
- net RD2: now also U1.88 (IO2_88); no longer U1.5 (IO1_5)
- net RD3: now also U1.89 (IO2_89); no longer U1.6 (IO1_6)
- net RD4: now also U1.90 (IO2_90); no longer U1.7 (IO1_7)
- net RD5: now also U1.91 (IO2_91); no longer U1.8 (IO1_8)
- net RD6: now also U1.92 (IO2_92); no longer U1.12 (IO1_12/GCLK0)
- net RD7: now also U1.99 (IO2_99); no longer U1.14 (IO1_14/GCLK1)
- net RDMAin: now also U1.48 (IO1_48), U5.12 (B6); no longer U1.49 (IO1_49), U5.11 (B7)
- net RDMAout: now also U1.18 (IO1_18), U18.1 (~OE~); no longer U1.20 (IO1_20)
- net RINTin: now also U1.49 (IO1_49), U5.11 (B7); no longer U1.48 (IO1_48), U5.12 (B6)
- net RINTout: now also U1.20 (IO1_20), U19.1 (~OE~); no longer U1.21 (IO1_21)
- net RR~W~out: now also U1.33 (IO1_33), U20.2 (A); no longer U1.28 (IO1_28)
- net R~W~: now also R1.1
- net SDQML: no longer U1.95 (IO2_95)
- net TCK: now also R29.1
- net TMS: now also R28.2
- net Vin: now also D1.1 (K)
- net ~DMA~: now also R23.1
- net ~INH~: now also R27.1
- net ~IRQ~: now also R20.1
- net ~Menu~: now also R19.2, R30.1; no longer U1.98 (IO2_98)
- net ~NMI~: now also R21.1
- net ~PreBOD~: now also U1.96 (IO2_96); no longer U1.97 (IO2_97)
- net ~RDY~: now also R24.1
- net ~RES~: now also R22.1; no longer R5.1, U7.1
- net at R3.2, R5.2, R7.1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: now also C38.1; no longer C39.1
- net at R4.2, R6.1, U7.2 (-)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: now also C39.1; no longer C38.1
- net at C6.1, D2.1 (K), FB1.2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: now also D1.2 (A)
- removed net A~OE~: U1.96 (IO2_96), U4.19 (~OE~), U9.19 (~OE~)
- net DET: no longer names the net of J3.3
- removed net D~OE~: U1.17 (IO1_17), U6.19 (~OE~)
- net RB0 renamed SA10
- net RB1 renamed SA9
- net RB10 renamed SA7
- net RB11 renamed SA1
- net RB2 renamed SBA1
- net RB3 renamed SA11
- net RB4 renamed SBA0
- net RB5 renamed SA12
- net RB6 renamed MOSI
- net MOSI: now also J5.8 (Pin_8), R19.1, U3.5 (DI/IO0)
- net RB7 renamed SA5
- net RB8 renamed SA2
- net RB9 renamed SA8
- net RPHI1 renamed RPHI0
- new net: R22.2, U14.4 (Y)
- new net: R20.2, U11.4 (Y)
- new net: R21.2, U12.4 (Y)
- new net: R23.2, U15.4 (Y)
- new net: R24.2, U17.4 (Y)
- new net: R25.2, U18.4 (Y)
- new net: R26.2, U19.4 (Y)
- new net: R1.2, U20.4 (Y)
- new net: J5.6 (Pin_6), R31.2
- new net: R27.2, U22.4 (Y)
- new net FCK: R31.1, U1.12 (IO1_12/GCLK0), U3.6 (CLK)
- new net FD2: J5.5 (Pin_5), RN5.1 (R1.1), U3.3 (~WP~/IO2)
- new net FD3: J5.4 (Pin_4), RN5.4 (R4.1), U3.7 (~HLD~/IO3)
- new net F~CS~: J5.1 (Pin_1), U1.5 (IO1_5), U3.1 (~CS~)
- new net MISO: J5.3 (Pin_3), U1.16 (IO1_16), U3.2 (DO/IO1)
- new net RDY~OE~: U1.28 (IO1_28), U17.1 (~OE~)
- new net RES~OE~: U1.30 (IO1_30), U14.1 (~OE~)
- new net ~BOD~: R2.2, R5.1, U1.95 (IO2_95), U7.1
- no-connect marks 22 -> 18
Other:
- note added: "(-) is 1.03125V\n~BOD~ at 4.43V\n~PreBOD~ at 4.78V"
- note removed: "Reference input is 1.03125V\n~RES~ (+) input is 1.05V @ 4.2V\n~PreBOD~ (+) inpt is 1.0465V @ 4.5V\n 1.1628V @ 5.0V\n 1.2791V @ 5.5V"
- moved on the sheet: C1, C10, C11, C12, C13, C14, C15, C16, C18, C19, C2, C20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

Commit message: idk
Parts:
- added C17: 2u2, stdpads:C_0603, symbol Device:C_Small
- C39: value 1n -> 2u2; LCSC Part C1588 -> C23630
- C41: value 22n -> 2u2; LCSC Part C21122 -> C23630
- R18: value 22k -> 100k; LCSC Part C31850 -> C25803
- R19: value 1k -> 33k; LCSC Part C21190 -> C4216
Connections:
- net Vin: now also C17.1
- net at C39.1, R4.2, R6.1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: now also C17.2
Changed lines of the file:
@@
 $EndDescr
 $Sheet
-S 500  600  500  150
+S 750  650  500  150
 U 5D4D21A0
 F0 "Docs" 50
@@
 Text Label 900  6550 2    50   ~ 0
 FD2
-$Comp
-L Device:R_Small R19
-U 1 1 5FFDC1D7
-P 8300 5000
-F 0 "R19" V 8250 5000 50  0000 C BNN
-F 1 "1k" V 8350 5000 50  0000 C TNN
-F 2 "stdpads:R_0603" H 8300 5000 50  0001 C CNN
-F 3 "~" H 8300 5000 50  0001 C CNN
-F 4 "C21190" H 8300 5000 50  0001 C CNN "LCSC Part"
-	1    8300 5000
-	0    1    1    0
-$EndComp
 Connection ~ 7800 5000
 Wire Wire Line
@@
 P 7050 4750
 F 0 "R18" H 7100 4800 50  0000 L CNN
-F 1 "22k" H 7100 4700 50  0000 L CNN
+F 1 "100k" H 7100 4700 50  0000 L CNN
 F 2 "stdpads:R_0603" H 7050 4750 50  0001 C CNN
 F 3 "~" H 7050 4750 50  0001 C CNN
-F 4 "C31850" H 7050 4750 50  0001 C CNN "LCSC Part"
+F 4 "C25803" H 7050 4750 50  0001 C CNN "LCSC Part"
 	1    7050 4750
 	1    0    0    -1
@@
 	1    0    0    -1
 $EndComp
-$Comp
-L Device:C_Small C39
-U 1 1 5FFA952A
-P 4750 1300
-F 0 "C39" H 4842 1346 50  0000 L CNN
-F 1 "1n" H 4842 1255 50  0000 L CNN
-F 2 "stdpads:C_0603" H 4750 1300 50  0001 C CNN
-F 3 "~" H 4750 1300 50  0001 C CNN
-F 4 "C1588" H 4750 1300 50  0001 C CNN "LCSC Part"
-	1    4750 1300
-	1    0    0    -1
-$EndComp
 Wire Wire Line
 	4100 1150 4750 1150
@@
 Wire Wire Line
 	4350 1200 4350 950
-$Comp
-L Device:C_Small C38
-U 1 1 5FB5B1B9
-P 4350 1300
-F 0 "C38" H 4442 1346 50  0000 L CNN
-F 1 "22n" H 4442 1255 50  0000 L CNN
-F 2 "stdpads:C_0603" H 4350 1300 50  0001 C CNN
-F 3 "~" H 4350 1300 50  0001 C CNN
-F 4 "C21122" H 4350 1300 50  0001 C CNN "LCSC Part"
-	1    4350 1300
-	1    0    0    -1
-$EndComp
 Wire Wire Line
 	4350 1450 4350 1400
@@
 	3300 1050 3500 1050
 $Comp
-L Device:C_Small C41
-U 1 1 5FF9336A
-P 7050 5200
-F 0 "C41" H 7142 5246 50  0000 L CNN
-F 1 "22n" H 7142 5155 50  0000 L CNN
-F 2 "stdpads:C_0603" H 7050 5200 50  0001 C CNN
-F 3 "~" H 7050 5200 50  0001 C CNN
-F 4 "C21122" H 7050 5200 50  0001 C CNN "LCSC Part"
-	1    7050 5200
-	1    0    0    -1
-$EndComp
-Wire Wire Line
-	6750 5300 7050 5300
-Wire Wire Line
-	7050 5300 7400 5300
-Connection ~ 7050 5300
-$Comp
 L Device:R_Small R31
 U 1 1 60BD9796
@@
 Wire Wire Line
 	3400 4250 4150 4250
-Wire Bus Line
-	600  3750 600  4650
-Wire Bus Line
-	1800 4650 1800 5450
-Wire Bus Line
-	3300 1950 3300 4550
-Wire Bus Line
-	3300 4850 3300 5550
-Wire Bus Line
-	1800 2350 1800 4250
 $Comp
 L Device:C_Small C2
@@
 	1    0    0    -1
 $EndComp
+Wire Wire Line
+	5050 900  4750 900
+Connection ~ 5050 900
+$Comp
+L Device:C_Small C38
+U 1 1 5FB5B1B9
+P 4350 1300
+F 0 "C38" H 4442 1346 50  0000 L CNN
+F 1 "22n" H 4442 1255 50  0000 L CNN
+F 2 "stdpads:C_0603" H 4350 1300 50  0001 C CNN
+F 3 "~" H 4350 1300 50  0001 C CNN
+F 4 "C21122" H 4350 1300 50  0001 C CNN "LCSC Part"
+	1    4350 1300
+	1    0    0    -1
+$EndComp
+Wire Wire Line
+	6750 5300 7050 5300
+$Comp
+L Device:C_Small C41
+U 1 1 6070D634
+P 7050 5200
+F 0 "C41" H 7100 5250 50  0000 L CNN
+F 1 "2u2" H 7100 5150 50  0000 L CNN
+F 2 "stdpads:C_0603" H 7050 5200 50  0001 C CNN
+F 3 "~" H 7050 5200 50  0001 C CNN
+F 4 "C23630" H 7050 5200 50  0001 C CNN "LCSC Part"
+	1    7050 5200
+	1    0    0    -1
+$EndComp
+Connection ~ 7050 5300
+Wire Wire Line
+	7050 5300 7400 5300
+$Comp
+L Device:C_Small C39
+U 1 1 604926F4
+P 4750 1300
+F 0 "C39" H 4800 1350 50  0000 L CNN
+F 1 "2u2" H 4800 1250 50  0000 L CNN
+F 2 "stdpads:C_0603" H 4750 1300 50  0001 C CNN
+F 3 "~" H 4750 1300 50  0001 C CNN
+F 4 "C23630" H 4750 1300 50  0001 C CNN "LCSC Part"
+	1    4750 1300
+	1    0    0    -1
+$EndComp
+$Comp
+L Device:C_Small C17
+U 1 1 60492089
+P 4750 800
+F 0 "C17" H 4800 850 50  0000 L CNN
+F 1 "2u2" H 4800 750 50  0000 L CNN
+F 2 "stdpads:C_0603" H 4750 800 50  0001 C CNN
+F 3 "~" H 4750 800 50  0001 C CNN
+F 4 "C23630" H 4750 800 50  0001 C CNN "LCSC Part"
+	1    4750 800
+	1    0    0    -1
+$EndComp
+Text GLabel 4750 700  0    50   Input ~ 0
+Vin
+$Comp
+L Device:R_Small R19
+U 1 1 5FFDC1D7
+P 8300 5000
+F 0 "R19" V 8250 5000 50  0000 C BNN
+F 1 "33k" V 8350 5000 50  0000 C TNN
+F 2 "stdpads:R_0603" H 8300 5000 50  0001 C CNN
+F 3 "~" H 8300 5000 50  0001 C CNN
+F 4 "C4216" H 8300 5000 50  0001 C CNN "LCSC Part"
+	1    8300 5000
+	0    1    1    0
+$EndComp
+Wire Bus Line
+	3300 4850 3300 5550
+Wire Bus Line
+	600  3750 600  4650
+Wire Bus Line
+	1800 4650 1800 5450
+Wire Bus Line
+	1800 2350 1800 4250
+Wire Bus Line
+	3300 1950 3300 4550
 $EndSCHEMATC

Commit message: Works?
Parts:
- removed C17, C39, C41: 2u2, stdpads:C_0603, symbol Device:C_Small
- removed C38, C40: 22n, stdpads:C_0603, symbol Device:C_Small
- removed C5, C6: 10u, stdpads:C_0805, symbol Device:C_Small
- removed D1, D3: SS34, stdpads:D_SMA, symbol Device:D_Schottky_Small_ALT
- removed D2: SMBJ5.0A, stdpads:D_SMB, symbol Device:D_Zener_Small_ALT
- removed F1: nSMD050-16V, stdpads:BelFuse_1206, symbol Device:Polyfuse_Small
- removed FB1: GZ2012D101TF, stdpads:Murata_BLM21, symbol Device:Ferrite_Bead_Small
- removed J3: DC in, stdpads:BOOMELE_DC-005_DC_5.5-2.0MM, symbol Connector:Barrel_Jack_Switch
- removed Q1: AO3401A, stdpads:SOT-23, symbol Transistor_FET:AO3401A
- removed R1, R20, R21, R23, R24, R25, R26, R27: 33, stdpads:R_0603, symbol Device:R_Small
- removed R10, R15, R16, R2, R4: 2k2, stdpads:R_0603, symbol Device:R_Small
- removed R11: 330, stdpads:R_0603, symbol Device:R_Small
- removed R12: 1k, stdpads:R_0805, symbol Device:R_Small
- removed R13: DNP, stdpads:R_0805, symbol Device:R_Small
- removed R14, R17, R6: 1k, stdpads:R_0603, symbol Device:R_Small
- removed R18: 100k, stdpads:R_0603, symbol Device:R_Small
- removed R19: 33k, stdpads:R_0603, symbol Device:R_Small
- removed R3: 2k7, stdpads:R_0603, symbol Device:R_Small
- removed R30, R5, R8: 1M, stdpads:R_0603, symbol Device:R_Small
- removed R7: 820, stdpads:R_0603, symbol Device:R_Small
- removed R9: 1k2, stdpads:R_0603, symbol Device:R_Small
- removed RN4: 4x10k, stdpads:R4_0402, symbol Device:R_Pack04
- removed U10, U7: LM393D, stdpads:SOIC-8_3.9mm, symbol Comparator:LM393
- removed U11, U12, U15, U17, U18, U19, U20, U22: 74LVC1G125GW, stdpads:SOT-353, symbol GW_Logic:741G125GW
Connections:
- net DMAout is gone; now on net DMAin: J1.24 (Pin_24)
- net INTout is gone; now on net INTin: J1.23 (Pin_23)
- net Vin is gone; now on net +5V: C7.1, C8.1, U8.3 (Vin)
- net +3V3: now also U9.1 (AtoB)
- net Adir: no longer U9.1 (AtoB)
- no-connect marks 18 -> 14
Other:
- note removed: "(-) is 1.03125V\n~BOD~ at 4.43V\n~PreBOD~ at 4.78V"

Commit message: idk
Parts:
- removed C36, C37, C8: 10u, stdpads:C_0805, symbol Device:C_Small
- removed C9: 2u2, stdpads:C_0603, symbol Device:C_Small
- added C5: 2u2, stdpads:C_0603, symbol Device:C_Small
- added SW1: FW, stdpads:SW_DIP_SPSTx02_Slide_DSHP02TS_P1.27mm, symbol Switch:SW_DIP_x02
- U3: LCSC Part C97521 -> C164122
Connections:
- net +3V3: now also U4.1 (AtoB), C5.1
- net DMAin: no longer U5.8 (A6)
- net GND: now also U5.8 (A6), U5.9 (A7), C5.2, SW1.1, SW1.2
- net INTin: no longer U5.9 (A7)
- net Adir: no longer names the net of U1.19 (IO1_19)
- net Adir: no longer U4.1 (AtoB)
- net DMA~OE~: no longer names the net of U1.21 (IO1_21)
- net INH~OE~: no longer names the net of U1.27 (IO1_27)
- net IRQ~OE~: no longer names the net of U1.29 (IO1_29)
- net NMI~OE~: no longer names the net of U1.26 (IO1_26)
- net RDMAin: no longer names the net of U5.12 (B6)
- net RDMAin: no longer U1.48 (IO1_48)
- net RDMAout: no longer names the net of U1.18 (IO1_18)
- net RDY~OE~: no longer names the net of U1.28 (IO1_28)
- net RINTin: no longer names the net of U5.11 (B7)
- net RINTin: no longer U1.49 (IO1_49)
- net RINTout: no longer names the net of U1.20 (IO1_20)
- net RR~W~out: no longer names the net of U1.33 (IO1_33)
- net ~BOD~ renamed FW1
- net FW1: now also SW1.4
- net ~PreBOD~ renamed FW0
- net FW0: now also SW1.3
- no-connect marks 14 -> 16
Other:
- moved on the sheet: C1, C12, C13, C14, C15, C16, C18, C19, C2, C20, C21, C22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
