File: Hardware/MAX/GR8RAM.kicad_sch (KiCad schematic)
At the start: 69 parts, among them J1 AppleIIBus, J2 JTAG, J4 JTAG, J5 JTAG, SW1 FW, U1 EPM240T100C5N, U13 25M, U14 74LVC1G125GW, U16 74LVC1G125GW, U2 W9825, U3 W25Q128JVSIQ, U4 74AHC245PW, U5 74AHC245PW, U6 74AHC245PW, U8 XC6206P332MR, U9 74AHC245PW

Commit message: rev. B boards almost done
Parts:
- removed C43, C44: 2u2, stdpads:C_0603, symbol Device:C_Small
- removed H6: (no value), stdpads:PasteHole_1.152mm_NPTH, symbol Mechanical:MountingHole
- removed J4: JTAG, Connector_IDC:IDC-Header_2x05_P2.54mm_Vertical, symbol Connector_Generic:Conn_02x05_Odd_Even
- removed R22, R31: 33, stdpads:R_0603, symbol Device:R_Small
- removed R28, R29: 22k, stdpads:R_0603, symbol Device:R_Small
- removed RN1, RN2, RN3: 4x33, stdpads:R4_0402, symbol Device:R_Pack04
- removed RN5: 4x10k, stdpads:R4_0402, symbol Device:R_Pack04
- added C17, C39, C40, C6: 2u2, stdpads:C_0603, symbol Device:C_Small
- added C36, C37, C38: 10u, stdpads:C_0805, symbol Device:C_Small
- added C41, C8, C9: 22p, stdpads:C_0603, symbol Device:C_Small
- added J3: microUSB, stdpads:USB_Micro-B_Amphenol_10118192-0001, symbol Connector:USB_B_Micro
- added R1: 0, stdpads:R_0805, symbol Device:R_Small
- added R10: 22, stdpads:R_0603, symbol Device:R_Small
- added R11: DNP, stdpads:R_0603, symbol Device:R_Small
- added R12, R13, R2, R3, R5, R9: 47, stdpads:R_0603, symbol Device:R_Small
- added R4, R6, R7, R8: 10k, stdpads:R_0603, symbol Device:R_Small
- added U10: AP2127K-1.8TRG1, stdpads:SOT-23-5, symbol Regulator_Linear:AP2127K-1.8
- added U11: 74LVC1G125GW, stdpads:SOT-353, symbol GW_Logic:741G125GW
- added U7: CH340G, stdpads:SOIC-16_3.9mm, symbol Interface_USB:CH340G
- added Y1: 12M, stdpads:Crystal_SMD_3225-4Pin_3.2x2.5mm, symbol Device:Crystal_GND24_Small
- J5: value JTAG -> Flash
- U1: symbol GW_PLD:EPM240T100 -> GW_PLD:5M240ZT100
- U3: LCSC Part C164122 -> C97521
Connections:
- net Dr0 is gone; now on net SD0: U1.50 (IO1_50)
- net Dr1 is gone; now on net SD1: U1.47 (IO1_47)
- net Dr2 is gone; now on net SD2: U1.56 (IO2_56)
- net Dr3 is gone; now on net SD3: U1.55 (IO2_55)
- net Dr4 is gone; now on net SD4: U1.51 (IO1_51)
- net Dr5 is gone; now on net SD5: U1.52 (IO2_52)
- net Dr6 is gone; now on net SD6: U1.53 (IO2_53)
- net Dr7 is gone; now on net SD7: U1.54 (IO2_54)
- net +3V3: now also C17.1, C36.1, C39.1, C40.1, R1.1, R4.2, R6.2, R7.1, U10.1 (VIN), U10.3 (EN), U11.5 (Vcc), U7.10 (~{DSR}), U7.11 (~{RI}), U7.16 (VCC), U7.3 (RXD), U7.4 (V3); no longer C19.1, C20.1, U1.13 (VCCINT), U1.63 (VCCINT)
- net ACLK: now also R3.1
- net FCK: now also R9.1
- net FD2: now also R4.1
- net FD3: now also R6.1
- net GND: now also U1.1 (GND), C17.2, C36.2, C37.2, C38.2, C39.2, C40.2, C41.2, C6.2, C8.2, C9.2, J3.5 (GND), J3.6 (Shield), R8.2, U10.2 (GND), U11.2 (A), U11.3 (GND), U7.1 (GND), U7.12 (~{DCD}), U7.15 (R232), Y1.2, Y1.4
- net RA4: now also U1.33 (IO1_33); no longer U1.1 (IO2_1)
- net RCLK: now also R2.1
- net TCK: now also C41.1, R12.2, R5.2, R8.1; no longer J2.1 (Pin_1)
- net TDI: now also U7.13 (~{DTR})
- net TDO: now also U7.9 (~{CTS})
- net TMS: now also R7.2, U7.14 (~{RTS})
- net ~{IRQ}: now also R13.1
- net ~{RES}: now also R10.1, R11.1
- net at U16.4 (Y): now also R2.2, R3.2
- net at U14.4 (Y): now also R10.2, R11.2
- net at J5.6 (Pin_6): now also R9.2
- net IRQ~{OE}: now reaches U1.28 (IO1_28)
- net IRQ~{OE}: now also U11.1 (~{OE})
- new net: J2.1 (Pin_1), R12.1
- new net: C9.1, U7.7 (XI), Y1.1
- new net: J3.3 (D+), U7.5 (UD+)
- new net: J3.2 (D-), U7.6 (UD-)
- new net: C8.1, U7.8 (XO), Y1.3
- new net: R13.2, U11.4 (Y)
- new net +1V8: C19.1, C20.1, C37.1, C38.1, R1.2, U1.13 (VCCINT), U1.63 (VCCINT), U10.5 (VOUT)
- new net USB5V: C6.1, J3.1 (VBUS)
- new net UTCK: R5.1, U7.2 (TXD)
- no-connect marks 16 -> 8
Other:
- removed sheet Docs
- moved on the sheet: C1, C10, C11, C12, C13, C14, C15, C16, C18, C19, C2, C20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
