File: Hardware/LCMXO2/GR8RAM.kicad_pcb (KiCad board)
At the start: 4 copper layers, 99.9 x 59.8 mm, 93 parts, among them J1 AppleIIBus, J2 JTAG, J3 microUSB, J5 Flash, SW1 FW, U1 LCMXO2-640-TG100, U10 AP2127K-1.2TRG1, U11 74LVC1G125GW, U13 25M, U14 74LVC1G125GW, U2 W9825, U3 W25Q128JVSIQ, U4 74AHC245PW, U5 74AHC245PW, U6 74AHC245PW, U7 CH340G, U8 XC6206P332MR, U9 74AHC245PW, Y1 12M

Commit message: 1.0 RC
Parts:
- removed R10: 22, stdpads:R_0603
- removed R11: DNP, stdpads:R_0603
- removed R13: 47, stdpads:R_0603
- added R14: 2k2, stdpads:R_0603, F.Cu at (115.8, 118.7)
- added R16: 2k2, stdpads:R_0603, F.Cu at (118.8, 118.7)
- U11, U14: value 74LVC1G125GW -> 74AHCT1G125GW
- moved J2 0.55 mm to (47.5, 99.8)
- renumbered J3 to J2, J5 to J3, J2 to J4
Connections:
- C39 pad 1: +3V3 -> +5V
- C42 pad 1: +3V3 -> +5V
- U11 pad 4: Net-(U11-Y) -> /~{IRQ}
- U11 pad 5: +3V3 -> +5V
- U14 pad 4: Net-(U14-Y) -> /~{RES}
- U14 pad 5: +3V3 -> +5V
Routing:
- net +5V: track 40.0 -> 96.4 mm, vias 3 -> 11
- net +3V3: track 168.9 -> 162.8 mm, vias 129 -> 122
- net Net-(U14-Y): track 3.72 -> 0.00 mm
- net /~{IRQ}: track 14.6 -> 18.2 mm
- net Net-(U11-Y): track 2.27 -> 0.00 mm
- net /FW1: track 49.3 -> 47.7 mm
- net /FW0: track 51.5 -> 49.9 mm
- net /~{RES}: track 28.2 -> 26.8 mm
- net /RES~{OE}: track 35.2 -> 36.1 mm
- net /IRQ~{OE}: track 36.1 -> 37.0 mm
- net GND: track 217.0 -> 216.7 mm, vias 438 -> 442
Other:
- board text added: "!"
- board text added: "B10C"
- board text added: "JLCJLCJLC"
- board text added: "Toward Rear"
- board text removed: "B10B"

Commit message: idk
Parts:
- added R10: 47, stdpads:R_0603, F.Cu at (104.5, 115.6)
- added R11: 47, stdpads:R_0603, F.Cu at (106.0, 115.6)
- added R13: 47, stdpads:R_0603, F.Cu at (107.5, 115.6)
- added R21: 47, stdpads:R_0603, F.Cu at (109.0, 115.6)
- added R22: 47, stdpads:R_0603, F.Cu at (110.5, 115.6)
Connections:
- U5 pad 14: /R~{RES} -> Net-(U5-B4)
- U5 pad 15: /R~{IOSTRB} -> Net-(U5-B3)
- U5 pad 16: /RPHI0 -> Net-(U5-B2)
- U5 pad 17: /R~{DEVSEL} -> Net-(U5-B1)
- U5 pad 18: /R~{IOSEL} -> Net-(U5-B0)
Routing:
- net /RR~{W}in: track 19.6 -> 29.0 mm
- net /R~{IOSEL}: track 18.9 -> 13.8 mm
- net Net-(U5-B0): track 0.00 -> 4.82 mm
- net Net-(U5-B1): track 0.00 -> 3.79 mm
- net /R~{DEVSEL}: track 19.0 -> 15.2 mm
- net Net-(U5-B4): track 0.00 -> 3.00 mm
- net Net-(U5-B2): track 0.00 -> 3.00 mm
- net /RPHI0: track 19.0 -> 16.3 mm
- net Net-(U5-B3): track 0.00 -> 2.65 mm
- net /R~{IOSTRB}: track 19.2 -> 17.4 mm
- net /R~{RES}: track 22.0 -> 21.2 mm
- net GND: vias 442 -> 441

Commit message: RC
Parts:
- added D1: Amber, stdpads:LED_0805, F.Cu at (107.4, 93.2)
- J3, J4: footprint Connector:Tag-Connect_TC2050-IDC-FP_2x05_P1.27mm_Vertical -> stdpads:Tag-Connect_TC2050-IDC-FP_2x05_P1.27mm_Vertical
- R12: value 47 -> DNP
- R18, R19, R7, R8: value 10k -> DNP
- R20: value 2k2 -> 220; footprint stdpads:R_0603 -> stdpads:R_0805
- U1: value LCMXO2-640-TG100 -> LCMXO2-640HC-4TG100C
- U2: value W9825 -> W9825G6KH-6
- U4, U5, U9: value 74AHC245PW -> 74LVC245APW
- moved R20 39.3 mm to (107.4, 95.3)
Connections:
- net /~{PROG} renamed /LED
- R20 pad 1: /~{JTAGEN} -> Net-(D1-A)
- R20 pad 2: GND -> +3V3
- U1 pad 82: /~{JTAGEN} -> GND
Routing:
- net /~{JTAGEN}: track 28.5 -> 0.00 mm, vias 2 -> 0
- net /LED: track 29.1 -> 53.2 mm, vias 2 -> 3
- net /RR~{W}in: track 29.0 -> 23.9 mm
- net Net-(D1-A): track 0.00 -> 2.10 mm
- net +3V3: track 162.7 -> 164.5 mm, vias 122 -> 123
- net /FW0: track 49.9 -> 50.8 mm
- net GND: track 216.7 -> 217.6 mm, vias 441 -> 446
- net /FW1: track 47.7 -> 48.4 mm
