File: Hardware/LCMXO2/GR8RAM.kicad_pcb (KiCad board)
At the start: 4 copper layers, 99.9 x 59.8 mm, 98 parts, among them J1 AppleIIBus, J2 microUSB, J3 Flash, J4 JTAG, SW1 FW, U1 LCMXO2-640HC-4TG100C, U10 AP2127K-1.2TRG1, U11 74AHCT1G125GW, U13 25M, U14 74AHCT1G125GW, U2 W9825G6KH-6, U3 W25Q128JVSIQ, U4 74LVC245APW, U5 74LVC245APW, U6 74AHC245PW, U7 CH340G, U8 XC6206P332MR, U9 74LVC245APW, Y1 12M

Commit message: RC
Parts:
- added C45: 2u2, stdpads:C_0603, F.Cu at (67.4, 119.8)
- added R15: 10k, stdpads:R_0603, F.Cu at (86.8, 113.2)
- added U12: 74AHCT245PW, stdpads:TSSOP-20_4.4x6.5mm_P0.65mm, F.Cu at (71.8, 122.0)
- moved J3 12.7 mm to (56.3, 120.9)
- moved J4 12.7 mm to (56.3, 120.9)
- moved R12 12.7 mm to (56.5, 114.7)
- moved R4 12.7 mm to (50.7, 124.4)
- moved R6 12.7 mm to (50.7, 121.3)
- renumbered R15 to R23
Connections:
- R18 pad 2: /~{INIT} -> ~{INIT}
- R23 pad 2: /Ddir -> /Dout~{OE}
- U1 pad 1: /Ddir -> /Dout~{OE}
- U1 pad 77: /~{INIT} -> ~{INIT}
- U6 pad 1: /Ddir -> +3V3
- U6 pad 19: GND -> ~{INIT}
Routing:
- net +5V: track 96.4 -> 182.1 mm, vias 11 -> 16
- net ~{INIT}: track 0.00 -> 58.4 mm, vias 0 -> 4
- net /Dout~{OE}: track 0.00 -> 25.6 mm, vias 0 -> 2
- net /~{INIT}: track 23.6 -> 0.00 mm, vias 2 -> 0
- net /Ddir: track 21.2 -> 0.00 mm, vias 2 -> 0
- net /D7: track 21.1 -> 39.9 mm, vias 1 -> 2
- net /RD7: track 44.7 -> 63.0 mm
- net /D6: track 19.3 -> 37.4 mm, vias 1 -> 2
- net /RD6: track 52.1 -> 68.9 mm
- net /D5: track 17.3 -> 33.1 mm, vias 1 -> 2
- net /RD5: track 51.5 -> 66.7 mm
- net /D4: track 15.5 -> 29.3 mm, vias 1 -> 2
- net /RD4: track 52.3 -> 66.0 mm
- net /RD3: track 53.1 -> 65.2 mm
- net /D3: track 14.0 -> 25.3 mm, vias 1 -> 2
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
Commit message: RC
Other:
- board text added: "JLCJLCJLCJLC"
- board text removed: "JLCJLCJLC"
Changed lines of the file:
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@@
     (effects (font (size 0.9525 0.9525) (thickness 0.2032)) (justify left))
   )
-  (gr_text "JLCJLCJLC" (at 92.8 101.4 90) (layer "F.SilkS")
+  (gr_text "JLCJLCJLCJLC" (at 121.2 103.05 90) (layer "F.SilkS")
     (effects (font (size 0.8128 0.8128) (thickness 0.2032)))
   )

Commit message: RC
Connections:
- U1 pad 82: GND -> +3V3
Routing:
- net GND: track 219.8 -> 218.2 mm, vias 420 -> 419
- net +3V3: track 167.9 -> 169.5 mm
Changed lines of the file:
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@@
   (title_block
     (title "GR8RAM (GW4205B) - LCMXO2-640 / LCMXO2-1200")
-    (date "2024-04-23")
+    (date "2024-05-20")
     (rev "1.0")
     (company "Garrett's Workshop")
@@
       (net 152 "/LED") (pinfunction "~{PROGRAM}/PT10D") (pintype "bidirectional"))
     (pad "82" smd roundrect (at -7.6625 -3 90) (size 0.3 1.475) (layers "F.Cu" "F.Paste" "F.Mask") (roundrect_rratio 0.25)
-      (net 2 "GND") (pinfunction "~{JTAGEN}/PT10C") (pintype "bidirectional"))
+      (net 70 "+3V3") (pinfunction "JTAGEN/PT10C") (pintype "bidirectional"))
     (pad "83" smd roundrect (at -7.6625 -2.5 90) (size 0.3 1.475) (layers "F.Cu" "F.Paste" "F.Mask") (roundrect_rratio 0.25)
       (net 52 "/RA2") (pinfunction "PT10B") (pintype "bidirectional"))
@@
   (segment (start 127.2 104.55) (end 127.45 104.3) (width 0.6) (layer "F.Cu") (net 2))
   (segment (start 67.4 120.55) (end 67.4 121.4) (width 0.6) (layer "F.Cu") (net 2))
-  (segment (start 86.3875 98.4) (end 87.3 98.4) (width 0.15) (layer "F.Cu") (net 2))
   (segment (start 98.05 111.15) (end 98.05 110.45) (width 0.5) (layer "F.Cu") (net 2))
   (segment (start 120.826 129.491) (end 120.777 129.54) (width 0.8) (layer "F.Cu") (net 2))
@@
   (segment (start 115.394 129.491) (end 115.443 129.54) (width 0.8) (layer "F.Cu") (net 2))
   (segment (start 110.8 103.3) (end 110.8 102.45) (width 0.6) (layer "F.Cu") (net 2))
-  (segment (start 87.3 98.4) (end 87.5 98.6) (width 0.15) (layer "F.Cu") (net 2))
   (segment (start 135.2 123.25) (end 135.2 122.3) (width 0.8) (layer "F.Cu") (net 2))
   (segment (start 132.75 118.7) (end 131.75 118.7) (width 0.8) (layer "F.Cu") (net 2))
@@
   (segment (start 112.9 103.05) (end 111.75 103.05) (width 0.45) (layer "F.Cu") (net 2))
   (segment (start 63.8175 99.9095) (end 63.8175 99.06) (width 0.5) (layer "F.Cu") (net 2))
-  (segment (start 87.65 98.75) (end 87.85 98.75) (width 0.15) (layer "F.Cu") (net 2))
   (segment (start 108.2 103.35) (end 108.2 104.2) (width 0.5) (layer "F.Cu") (net 2))
   (segment (start 135.46 128.27) (end 135.46 127.049) (width 0.762) (layer "F.Cu") (net 2))
   (segment (start 97.25 92.55) (end 97.05 92.35) (width 0.5) (layer "F.Cu") (net 2))
-  (segment (start 87.5 98.6) (end 87.65 98.75) (width 0.15) (layer "F.Cu") (net 2))
   (segment (start 126.45 94.15) (end 127.2 94.15) (width 0.8) (layer "F.Cu") (net 2))
   (segment (start 121.2 120.85) (end 121.2 120.05) (width 0.5) (layer "F.Cu") (net 2))
@@
   (via (at 50.75 96.7) (size 0.5) (drill 0.3) (layers "F.Cu" "B.Cu") (net 2))
   (via (at 111.55 126.1) (size 0.5) (drill 0.3) (layers "F.Cu" "B.Cu") (net 2))
-  (via (at 87.85 98.75) (size 0.5) (drill 0.3) (layers "F.Cu" "B.Cu") (net 2))
   (via (at 117.983 86.9315) (size 0.5) (drill 0.3) (layers "F.Cu" "B.Cu") (net 2))
   (via (at 84.6 124.95) (size 0.5) (drill 0.3) (layers "F.Cu" "B.Cu") (net 2))
@@
   (segment (start 90.05 110.1) (end 89.9 110.25) (width 0.3) (layer "F.Cu") (net 70))
   (segment (start 140.1 120.4) (end 141.1 120.4) (width 0.8) (layer "F.Cu") (net 70))
+  (segment (start 86.3875 98.4) (end 85.5 98.4) (width 0.15) (layer "F.Cu") (net 70))
   (segment (start 50.7365 123.5585) (end 50.7365 122.809) (width 0.15) (layer "F.Cu") (net 70))
   (segment (start 90.05 109.0625) (end 90.05 110.1) (width 0.3) (layer "F.Cu") (net 70))
@@
   (segment (start 124.4 107.05) (end 125.55 107.05) (width 0.45) (layer "F.Cu") (net 70))
   (segment (start 124.4 90.75) (end 125.25 90.75) (width 0.6) (layer "F.Cu") (net 70))
+  (segment (start 85.5 98.4) (end 85 97.9) (width 0.15) (layer "F.Cu") (net 70))
   (segment (start 62.103 101.408) (end 62.103 100.0125) (width 0.5) (layer "F.Cu") (net 70))
   (segment (start 135.2 125.15) (end 134.25 125.15) (width 0.8) (layer "F.Cu") (net 70))
