File: Hardware/LCMXO2/GR8RAM.kicad_sch (KiCad schematic)
At the start: 91 parts, among them J1 AppleIIBus, J2 JTAG, J3 microUSB, J5 Flash, SW1 FW, U1 LCMXO2-640-TG100, U10 AP2127K-1.2TRG1, U11 74LVC1G125GW, U13 25M, U14 74LVC1G125GW, U2 W9825, U3 W25Q128JVSIQ, U4 74AHC245PW, U5 74AHC245PW, U6 74AHC245PW, U7 CH340G, U8 XC6206P332MR, U9 74AHC245PW, Y1 12M

Commit message: 1.0 RC
Parts:
- removed R10: 22, stdpads:R_0603, symbol Device:R_Small
- removed R11: DNP, stdpads:R_0603, symbol Device:R_Small
- removed R13: 47, stdpads:R_0603, symbol Device:R_Small
- added R14, R16: 2k2, stdpads:R_0603, symbol Device:R_Small
- R15, R20: LCSC Part (none) -> C4190
- U11, U14: value 74LVC1G125GW -> 74AHCT1G125GW; LCSC Part C12519 -> C12495
- renumbered J3 to J2, J5 to J3, J2 to J4
Connections:
- net +3V3: now also R14.1, R16.1; no longer C39.1, C42.1, U11.5 (Vcc), U14.5 (Vcc)
- net +5V: now also C39.1, C42.1, U11.5 (Vcc), U14.5 (Vcc)
- net IRQ~{OE}: now also R16.2
- net RES~{OE}: now also R14.2
- net ~{IRQ}: now also U11.4 (Y)
- net ~{RES}: now also U14.4 (Y)
Other:
- title: GR8RAM -> GR8RAM (GW4205B) - LCMXO2-640 / LCMXO2-1200
- moved on the sheet: C17, C39, R15, R2, U11

Commit message: idk
Parts:
- added R10, R11, R13, R21, R22: 47, stdpads:R_0603, symbol Device:R_Small
Connections:
- net RPHI0: now also R13.1; no longer U5.16 (B2)
- net R~{DEVSEL}: now also R11.1; no longer U5.17 (B1)
- net R~{IOSEL}: now also R10.1; no longer U5.18 (B0)
- net R~{IOSTRB}: now also R21.1; no longer U5.15 (B3)
- net R~{RES}: now also R22.1; no longer U5.14 (B4)
- new net: R22.2, U5.14 (B4)
- new net: R21.2, U5.15 (B3)
- new net: R13.2, U5.16 (B2)
- new net: R11.2, U5.17 (B1)
- new net: R10.2, U5.18 (B0)
Other:
- moved on the sheet: U5

Commit message: RC
Parts:
- added D1: Amber, stdpads:LED_0805, symbol Device:LED_Small_ALT
- J3, J4: footprint Connector:Tag-Connect_TC2050-IDC-FP_2x05_P1.27mm_Vertical -> stdpads:Tag-Connect_TC2050-IDC-FP_2x05_P1.27mm_Vertical
- R12: value 47 -> DNP; LCSC Part C23182 -> (none)
- R18, R19, R7, R8: value 10k -> DNP; LCSC Part C25804 -> (none)
- R20: value 2k2 -> 220; footprint stdpads:R_0603 -> stdpads:R_0805; LCSC Part C4190 -> C17557
- U1: value LCMXO2-640-TG100 -> LCMXO2-640HC-4TG100C; LCSC Part (none) -> C1519051
- U10: LCSC Part C151375 -> C151376
- U2: value W9825 -> W9825G6KH-6
- U4, U5, U9: value 74AHC245PW -> 74LVC245APW; LCSC Part C5516 -> C6082
Connections:
- net +3V3: now also R20.2
- net GND: now also U1.82 (~{JTAGEN}/PT10C); no longer R20.2
- net ~{JTAGEN}: no longer names the net of R20.1
- net ~{JTAGEN}: now also D1.2 (A); no longer U1.82 (~{JTAGEN}/PT10C)
- net ~{PROG} renamed LED
- net LED: now also D1.1 (K)
Other:
- moved on the sheet: R17, R18, R19, U2, U3

Commit message: RC
Parts:
- added C45: 2u2, stdpads:C_0603, symbol Device:C_Small
- added R23: 2k2, stdpads:R_0603, symbol Device:R_Small
- added U12: 74AHCT245PW, stdpads:TSSOP-20_4.4x6.5mm_P0.65mm, symbol GW_Logic:74245
- R15: value 2k2 -> 10k; LCSC Part C4190 -> C25804
Connections:
- net +3V3: now also U6.1 (AtoB), R23.1
- net +5V: now also C45.1, U12.20 (Vcc)
- net D0: now also U12.9 (A7)
- net D1: now also U12.8 (A6)
- net D2: now also U12.7 (A5)
- net D3: now also U12.6 (A4)
- net D4: now also U12.5 (A3)
- net D5: now also U12.4 (A2)
- net D6: now also U12.3 (A1)
- net D7: now also U12.2 (A0)
- net GND: now also C45.2, U12.1 (AtoB), U12.10 (GND); no longer U6.19 (~{OE})
- net RD0: now also U12.11 (B7)
- net RD1: now also U12.12 (B6)
- net RD2: now also U12.13 (B5)
- net RD3: now also U12.14 (B4)
- net RD4: now also U12.15 (B3)
- net RD5: now also U12.16 (B2)
- net RD6: now also U12.17 (B1)
- net RD7: now also U12.18 (B0)
- net ~{INIT}: now also R15.2, U6.19 (~{OE})
- removed net Ddir: R15.2, U1.1 (PL2A), U6.1 (AtoB)
- new net Dout~{OE}: R23.2, U1.1 (PL2A), U12.19 (~{OE})
Other:
- moved on the sheet: D1, J3, R14, R16, R17, R18, R19, R2, R20, R3, R9, SW1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

Commit message: RC
Connections:
- net +3V3: now also U1.82 (JTAGEN/PT10C)
- net GND: no longer U1.82 (~{JTAGEN}/PT10C)
Changed lines of the file:
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@@
   (title_block
     (title "GR8RAM (GW4205B) - LCMXO2-640 / LCMXO2-1200")
-    (date "2024-04-23")
+    (date "2024-05-20")
     (rev "1.0")
     (company "Garrett's Workshop")
@@
     )
   )
+  (symbol (lib_name "+3V3_1") (lib_id "power:+3V3") (at 161.29 90.17 0) (unit 1)
+    (in_bom yes) (on_board yes) (dnp no)
+    (property "Reference" "#PWR030" (at 161.29 93.98 0)
+      (effects (font (size 1.27 1.27)) hide)
+    )
+    (property "Value" "+3V3" (at 161.29 86.36 0)
+      (effects (font (size 1.27 1.27)))
+    )
+    (property "Footprint" "" (at 161.29 90.17 0)
+      (effects (font (size 1.27 1.27)) hide)
+    )
+    (property "Datasheet" "" (at 161.29 90.17 0)
+      (effects (font (size 1.27 1.27)) hide)
+    )
+    (pin "1")
+    (instances
+      (project "GR8RAM"
+        (path "/a29f8df0-3fae-4edf-8d9c-bd5a875b13e3"
+          (reference "#PWR030") (unit 1)
+        )
+      )
+    )
+  )
   (symbol (lib_id "Device:R_Small") (at 96.52 29.21 270) (unit 1)
     (in_bom yes) (on_board yes) (dnp no)
@@
         )
       )
-    )
-  )
-  (symbol (lib_id "power:GND") (at 161.29 90.17 0) (mirror y) (unit 1)
-    (in_bom yes) (on_board yes) (dnp no)
-    (property "Reference" "#PWR030" (at 161.29 96.52 0)
-      (effects (font (size 1.27 1.27)) hide)
-    )
-    (property "Value" "GND" (at 161.29 93.98 0)
-      (effects (font (size 1.27 1.27)))
-    )
-    (property "Footprint" "" (at 161.29 90.17 0)
-      (effects (font (size 1.27 1.27)) hide)
-    )
-    (property "Datasheet" "" (at 161.29 90.17 0)
-      (effects (font (size 1.27 1.27)) hide)
-    )
-    (pin "1")
-    (instances
-      (project "GR8RAM"
-        (path "/a29f8df0-3fae-4edf-8d9c-bd5a875b13e3"
-          (reference "#PWR030") (unit 1)
-        )
-      )

Commit message: dip switch stuff
Parts:
- added R24: 47, stdpads:R_0603, symbol Device:R_Small
- added R25, R26, R27: 10k, stdpads:R_0603, symbol Device:R_Small
- SW1: footprint stdpads:SW_DIP_SPSTx02_Slide_DSHP02TS_P1.27mm -> stdpads:SW_DIP_SPSTx03_Slide_DSHP03TS_P1.27mm; symbol Switch:SW_DIP_x02 -> Switch:SW_DIP_x03
Connections:
- net +3V3: now also R25.2, R26.2, R27.2
- net FW0: now also SW1.4, R26.1; no longer SW1.3
- net FW1: now also SW1.5, R25.1; no longer SW1.4
- net GND: now also SW1.3
- net RD0: now also R24.2
- new net ~{RESTORE}: R24.1, R27.1, SW1.6

Commit message: Another board RC
Parts:
- R24: value 47 -> 2k2; LCSC Part C23182 -> C4190
Connections:
- net RCLKout is gone; now on net RCLK: R2.2, U1.39 (PB10D/PCLKC2_1)
- net SA0 is gone; now on net RA0: U1.54 (PR7A), U2.23 (A0)
- net SA1 is gone; now on net RA1: U1.59 (PR6B), U2.24 (A1)
- net SA10 is gone; now on net RA10: U1.47 (PB14), U2.22 (A10)
- net SA11 is gone; now on net RA11: U1.45 (PB14A), U2.35 (A11)
- net SA12 is gone; now on net RA12: U1.42 (PB12C), U2.36 (A12)
- net SA2 is gone; now on net RA2: U1.58 (PR6C), U2.25 (A2)
- net SA3 is gone; now on net RA3: U1.60 (PR6A), U2.26 (A3)
- net SA4 is gone; now on net RA4: U1.51 (PR7D), U2.29 (A4)
- net SA5 is gone; now on net RA5: U1.52 (PR7C), U2.30 (A5)
- net SA6 is gone; now on net RA6: U1.62 (PCLKC1_0/PR5D), U2.31 (A6)
- net SA7 is gone; now on net RA7: U1.57 (PR6D), U2.32 (A7)
- net SA8 is gone; now on net RA8: U1.53 (PR7B), U2.33 (A8)
- net SA9 is gone; now on net RA9: U1.49 (PB14D/SI/SISPI), U2.34 (A9)
- net SD0 is gone; now on net RD0: U1.25 (PL7D), U2.2 (DQ0), U2.53 (DQ15)
- net SD1 is gone; now on net RD1: U1.24 (PL7C), U2.4 (DQ1), U2.51 (DQ14)
- net SD2 is gone; now on net RD2: U1.21 (PL7B/PCLKC3_0), U2.5 (DQ2), U2.50 (DQ13)
- net SD3 is gone; now on net RD3: U1.27 (PB4A/CSSPIN), U2.48 (DQ12), U2.7 (DQ3)
- net SD4 is gone; now on net RD4: U1.28 (PB4B), U2.47 (DQ11), U2.8 (DQ4)
- net SD5 is gone; now on net RD5: U1.29 (PB4C), U2.10 (DQ5), U2.45 (DQ10)
- net SD6 is gone; now on net RD6: U1.30 (PB4D), U2.11 (DQ6), U2.44 (DQ9)
- net SD7 is gone; now on net RD7: U1.31 (PB6A/MCLK/CCLK), U2.13 (DQ7), U2.42 (DQ8)
- net RA0: no longer U1.74 (PR2B), U4.18 (B0)
- net RA1: no longer U1.78 (PT11A), U4.17 (B1)
- net RA10: no longer U1.3 (PL2C/PCLKT3_2), U9.16 (B2)
- net RA11: no longer U1.8 (PL3B), U9.15 (B3)
- net RA12: no longer U1.9 (PL3C), U9.14 (B4)
- net RA2: no longer U1.83 (PT10B), U4.16 (B2)
- net RA3: no longer U1.84 (PT10A), U4.15 (B3)
- net RA4: no longer U1.4 (PL2D/PCLKC3_2), U4.14 (B4)
- net RA5: no longer U1.85 (SDA/PCLKC0_0/PT9D), U4.13 (B5)
- net RA6: no longer U1.86 (SCL/PCLKT0_0/PT9C), U4.12 (B6)
- net RA7: no longer U1.87 (PT9B/PCLKC0_1), U4.11 (B7)
- net RA8: no longer U1.99 (PT6A), U9.18 (B0)
- net RA9: no longer U1.2 (PL2B), U9.17 (B1)
- net RCLK: no longer R2.1, U2.38 (CLK)
- net RD0: no longer R24.2, U1.65 (PR5A), U12.11 (B7), U6.18 (B0)
- net RD1: no longer U1.66 (PR3D), U12.12 (B6), U6.17 (B1)
- net RD2: no longer U1.67 (PR3C), U12.13 (B5), U6.16 (B2)
- net RD3: no longer U1.68 (PR3B), U12.14 (B4), U6.15 (B3)
- net RD4: no longer U1.69 (PR3A), U12.15 (B3), U6.14 (B4)
- net RD5: no longer U1.70 (PR2D), U12.16 (B2), U6.13 (B5)
- net RD6: no longer U1.71 (PR2C), U12.17 (B1), U6.12 (B6)
- net RD7: no longer U1.75 (PR2A), U12.18 (B0), U6.11 (B7)
- net ACLK renamed CLKin
- net IRQ~{OE} renamed ~{IRQ}out
- net RA13 renamed BA13
- net RA14 renamed BA14
- net RA15 renamed BA15
- net RES~{OE} renamed ~{RES}out
- net RPHI0 renamed BPHI0
- net RR~{W}in renamed BR~{W}
- net R~{DEVSEL} renamed B~{DEVSEL}
- net R~{IOSEL} renamed B~{IOSEL}
- net R~{IOSTRB} renamed B~{IOSTRB}
- net R~{RES} renamed B~{RES}
- net SBA0 renamed RBA0
- net SBA1 renamed RBA1
- net SCKE renamed RCKE
- net SDQMH renamed DQMH
- net SDQML renamed DQML
- net S~{CAS} renamed ~{CAS}
- net S~{CS} renamed R~{CS}
- net S~{RAS} renamed ~{RAS}
- net S~{WE} renamed R~{WE}
- new net BA0: U1.74 (PR2B), U4.18 (B0)
- new net BA1: U1.78 (PT11A), U4.17 (B1)
- new net BA10: U1.3 (PL2C/PCLKT3_2), U9.16 (B2)
- new net BA11: U1.8 (PL3B), U9.15 (B3)
- new net BA12: U1.9 (PL3C), U9.14 (B4)
- new net BA2: U1.83 (PT10B), U4.16 (B2)
- new net BA3: U1.84 (PT10A), U4.15 (B3)
- new net BA4: U1.4 (PL2D/PCLKC3_2), U4.14 (B4)
- new net BA5: U1.85 (SDA/PCLKC0_0/PT9D), U4.13 (B5)
- new net BA6: U1.86 (SCL/PCLKT0_0/PT9C), U4.12 (B6)
- new net BA7: U1.87 (PCLKC0_1/PT9B), U4.11 (B7)
- new net BA8: U1.99 (PT6A), U9.18 (B0)
- new net BA9: U1.2 (PL2B), U9.17 (B1)
- new net BD0: R24.2, U1.65 (PR5A), U12.11 (B7), U6.18 (B0)
- new net BD1: U1.66 (PR3D), U12.12 (B6), U6.17 (B1)
- new net BD2: U1.67 (PR3C), U12.13 (B5), U6.16 (B2)
- new net BD3: U1.68 (PR3B), U12.14 (B4), U6.15 (B3)
- new net BD4: U1.69 (PR3A), U12.15 (B3), U6.14 (B4)
- new net BD5: U1.70 (PR2D), U12.16 (B2), U6.13 (B5)
- new net BD6: U1.71 (PR2C), U12.17 (B1), U6.12 (B6)
- new net BD7: U1.75 (PR2A), U12.18 (B0), U6.11 (B7)
- new net RCLKr: R2.1, U2.38 (CLK)
- no-connect marks 8 -> 9

Commit message: fix bom
Parts:
- H1, H2, H3, H4, H5: value (none) -> ~
- R14, R16, R23, R24: value 2k2 -> 3k3; LCSC Part C4190 -> C22978
- R15: value 10k -> 3k3; LCSC Part C25804 -> C22978
- R3: value 47 -> DNP; LCSC Part C23182 -> (none)
- SW1: LCSC Part C319052 -> C319051
- U10: value AP2127K-1.2TRG1 -> DNP; LCSC Part C151376 -> (none)
- U12: LCSC Part C5516 -> C173388
- U13: value 25M -> DNP; LCSC Part C669088 -> (none)
- U6: value 74AHC245PW -> 74LVC245APW; LCSC Part C5516 -> C6082
Connections:
- net +3V3: now also U1.11 ((VccIO3))
