File: Hardware/LCMXO2/GR8RAM.kicad_sch (KiCad schematic)
At the start: 103 parts, among them J1 AppleIIBus, J2 microUSB, J3 Flash, J4 JTAG, SW1 FW, U1 LCMXO2-640HC-4TG100C, U10 DNP, U11 74AHCT1G125GW, U12 74AHCT245PW, U13 DNP, U14 74AHCT1G125GW, U2 W9825G6KH-6, U3 W25Q128JVSIQ, U4 74LVC245APW, U5 74LVC245APW, U6 74LVC245APW, U7 CH340G, U8 XC6206P332MR, U9 74LVC245APW, Y1 12M

Commit message: Update PCB text, etc
Connections:
- net ~{INIT} renamed Din~{OE}
Other:
- moved on the sheet: R15, R2, R23
Changed lines of the file:
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@@
 	)
 	(bus_entry
-		(at 86.36 41.91)
-		(size 2.54 2.54)
-		(stroke
-			(width 0)
-			(type default)
-		)
-	)
-	(bus_entry
 		(at 83.82 80.01)
 		(size -2.54 2.54)
@@
 	(wire
 		(pts
-			(xy 113.03 187.96) (xy 113.03 190.5)
+			(xy 113.03 185.42) (xy 113.03 187.96)
 		)
 		(stroke
@@
 	(wire
 		(pts
-			(xy 105.41 175.26) (xy 97.79 175.26)
+			(xy 105.41 172.72) (xy 97.79 172.72)
 		)
 		(stroke
@@
 	(wire
 		(pts
-			(xy 97.79 190.5) (xy 113.03 190.5)
+			(xy 97.79 187.96) (xy 113.03 187.96)
 		)
 		(stroke
@@
 	(wire
 		(pts
-			(xy 110.49 175.26) (xy 115.57 175.26)
+			(xy 110.49 172.72) (xy 115.57 172.72)
 		)
 		(stroke
@@
 	(wire
 		(pts
-			(xy 97.79 187.96) (xy 105.41 187.96)
+			(xy 97.79 185.42) (xy 105.41 185.42)
 		)
 		(stroke
@@
 	)
 	(label "RCLKr"
-		(at 115.57 175.26 180)
+		(at 115.57 172.72 180)
 		(effects
 			(font
@@
 	)
 	(label "Din~{OE}"
-		(at 97.79 187.96 0)
+		(at 97.79 185.42 0)
 		(effects
 			(font
@@
 	)
 	(label "Dout~{OE}"
-		(at 97.79 190.5 0)
+		(at 97.79 187.96 0)
 		(effects
 			(font
@@
 	)
 	(label "RCLK"
-		(at 97.79 175.26 0)
+		(at 97.79 172.72 0)
 		(effects
 			(font
@@
 		)
 	)
-	(global_label "~{INIT}"
-		(shape input)
-		(at 161.29 97.79 0)
-		(fields_autoplaced yes)
-		(effects
-			(font
-				(size 1.27 1.27)
-			)
-			(justify left)
-		)
-		(property "Intersheetrefs" "${INTERSHEET_REFS}"
-			(at 167.1287 97.79 0)
-			(effects
-				(font
-					(size 1.27 1.27)
-				)
-				(justify left)
-				(hide yes)
-			)
-		)
-	)
 	(symbol
 		(lib_id "Device:C_Small")
@@
 	(symbol
 		(lib_id "Device:R_Small")
-		(at 107.95 175.26 270)
+		(at 107.95 172.72 270)
 		(unit 1)
 		(exclude_from_sim no)
@@
 		(dnp no)
 		(property "Reference" "R2"
-			(at 107.95 171.45 90)
+			(at 107.95 168.91 90)
 			(effects
 				(font
@@
 		)
 		(property "Value" "47"
-			(at 107.95 173.99 90)
+			(at 107.95 171.45 90)
 			(effects
 				(font
@@
 		)
 		(property "Footprint" "stdpads:R_0603"
-			(at 107.95 175.26 0)
+			(at 107.95 172.72 0)
 			(effects
 				(font
@@
 		)
 		(property "Datasheet" ""
-			(at 107.95 175.26 0)
+			(at 107.95 172.72 0)
 			(effects
 				(font
@@
 		)
 		(property "Description" ""
-			(at 107.95 175.26 0)
+			(at 107.95 172.72 0)
 			(effects
 				(font
@@
 		)
 		(property "LCSC Part" "C23182"
-			(at 107.95 175.26 0)
+			(at 107.95 172.72 0)
 			(effects
 				(font
@@
 	(symbol
 		(lib_id "Device:R_Small")
-		(at 105.41 185.42 0)
+		(at 105.41 182.88 0)
 		(unit 1)
 		(exclude_from_sim no)
@@
 		(dnp no)
 		(property "Reference" "R15"
-			(at 106.68 184.15 0)
+			(at 106.68 181.61 0)
 			(effects
 				(font
@@
 		)
 		(property "Value" "3k3"
-			(at 106.68 186.69 0)
+			(at 106.68 184.15 0)
 			(effects
 				(font
@@
 		)
 		(property "Footprint" "stdpads:R_0603"
-			(at 105.41 185.42 0)
+			(at 105.41 182.88 0)
 			(effects
 				(font
@@
 		)
 		(property "Datasheet" ""
-			(at 105.41 185.42 0)
+			(at 105.41 182.88 0)
 			(effects
 				(font
@@
 		)
 		(property "Description" ""
-			(at 105.41 185.42 0)
+			(at 105.41 182.88 0)
 			(effects
 				(font
@@
 		)
 		(property "LCSC Part" "C22978"
-			(at 105.41 185.42 0)
+			(at 105.41 182.88 0)
 			(effects
 				(font
@@
 	(symbol
 		(lib_id "Device:R_Small")
-		(at 113.03 185.42 0)
+		(at 113.03 182.88 0)
 		(unit 1)
 		(exclude_from_sim no)
@@
 		(dnp no)
 		(property "Reference" "R23"
-			(at 114.3 184.15 0)
+			(at 114.3 181.61 0)
 			(effects
 				(font
@@
 		)
 		(property "Value" "3k3"
-			(at 114.3 186.69 0)
+			(at 114.3 184.15 0)
 			(effects
 				(font
@@
 		)
 		(property "Footprint" "stdpads:R_0603"
-			(at 113.03 185.42 0)
+			(at 113.03 182.88 0)
 			(effects
 				(font
@@
 		)
 		(property "Datasheet" ""
-			(at 113.03 185.42 0)
+			(at 113.03 182.88 0)
 			(effects
 				(font
@@
 		)
 		(property "Description" ""
-			(at 113.03 185.42 0)
+			(at 113.03 182.88 0)
 			(effects
 				(font
@@
 		)
 		(property "LCSC Part" "C22978"
-			(at 113.03 185.42 0)
+			(at 113.03 182.88 0)
 			(effects
 				(font
@@
 	(symbol
 		(lib_id "power:+3V3")
-		(at 113.03 182.88 0)
+		(at 113.03 180.34 0)
 		(unit 1)
 		(exclude_from_sim no)
@@
 		(dnp no)
 		(property "Reference" "#PWR033"
-			(at 113.03 186.69 0)
+			(at 113.03 184.15 0)
 			(effects
 				(font
@@
 		)
 		(property "Value" "+3V3"
-			(at 113.03 179.07 0)
+			(at 113.03 176.53 0)
 			(effects
 				(font
@@
 		)
 		(property "Footprint" ""
-			(at 113.03 182.88 0)
+			(at 113.03 180.34 0)
 			(effects
 				(font
@@
 		)
 		(property "Datasheet" ""
-			(at 113.03 182.88 0)
+			(at 113.03 180.34 0)
 			(effects
 				(font
@@
 		)
 		(property "Description" ""
-			(at 113.03 182.88 0)
+			(at 113.03 180.34 0)
 			(effects
 				(font
@@
 	(symbol
 		(lib_id "power:+3V3")
-		(at 105.41 182.88 0)
+		(at 105.41 180.34 0)
 		(unit 1)
 		(exclude_from_sim no)
@@
 		(dnp no)
 		(property "Reference" "#PWR011"
-			(at 105.41 186.69 0)
+			(at 105.41 184.15 0)
 			(effects
 				(font
@@
 		)
 		(property "Value" "+3V3"
-			(at 105.41 179.07 0)
+			(at 105.41 176.53 0)
 			(effects
 				(font
@@
 		)
 		(property "Footprint" ""
-			(at 105.41 182.88 0)
+			(at 105.41 180.34 0)
 			(effects
 				(font
@@
 		)
 		(property "Datasheet" ""
-			(at 105.41 182.88 0)
+			(at 105.41 180.34 0)
 			(effects
 				(font
@@
 		)
 		(property "Description" ""
-			(at 105.41 182.88 0)
+			(at 105.41 180.34 0)
 			(effects
 				(font
